File: elec/layout/default/bmi088.kicad_pcb (KiCad board)
At the start: 2 copper layers, 225.7 x 100.8 mm, 0 parts

Commit message: initial layout
Parts:
- added C1: Multilayer Ceramic Capacitors MLCC - SMD/SMT 100nF 10V 0402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, lib:C0402, F.Cu at (156.6, 93.0)
- added C2: Multilayer Ceramic Capacitors MLCC - SMD/SMT 100nF 10V 0402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, lib:C0402, F.Cu at (161.7, 94.5)
- added U1: , lib:LGA-16_L4.5-W3.0-P0.50-BL, F.Cu at (159.1, 94.4)
Routing:
- net gnd: track 0.00 -> 10.6 mm
- net vcc: track 0.00 -> 8.55 mm
