File: elec/layout/default/bmi088.kicad_pcb (KiCad board)
At the start: 2 copper layers, 225.7 x 100.8 mm, 3 parts

Commit message: update layout
Parts:
- C1, C2: value Multilayer Ceramic Capacitors MLCC - SMD/SMT 100nF 10V 0402 RoHS -> 16V 100nF X7R ±10% 0402 Multilayer Ceramic Capacitors MLCC - SMD/SMT ROHS
Connections:
- U1 pad 14: csb1 -> vcc
- U1 pad 15: sdo2 -> sdo1
Routing:
- net vcc: track 8.55 -> 11.1 mm
Changed lines of the file:
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@@
   (net 1 "int1")
   (net 2 "sdo2")
-  (net 3 "csb1")
+  (net 3 "sdo1")
   (net 4 "int4")
   (net 5 "int3")
@@
         (effects (font (size 1 1) (thickness 0.15)))
     )
-    (fp_text value "Multilayer Ceramic Capacitors MLCC - SMD/SMT 100nF 10V 0402 RoHS" (at 0 1.16 90) (layer "F.Fab")
+    (fp_text value "16V 100nF X7R ±10% 0402  Multilayer Ceramic Capacitors MLCC - SMD/SMT ROHS" (at 0 1.16 90) (layer "F.Fab")
         (effects (font (size 1 1) (thickness 0.15)))
     )
@@
         (effects (font (size 1 1) (thickness 0.15)))
     )
-    (fp_text value "Multilayer Ceramic Capacitors MLCC - SMD/SMT 100nF 10V 0402 RoHS" (at 0 1.16 90) (layer "F.Fab")
+    (fp_text value "16V 100nF X7R ±10% 0402  Multilayer Ceramic Capacitors MLCC - SMD/SMT ROHS" (at 0 1.16 90) (layer "F.Fab")
         (effects (font (size 1 1) (thickness 0.15)))
     )
@@
       (net 4 "int4") (pintype "stereo"))
     (pad "14" smd rect (at 1.2 1 270) (size 0.25 0.8) (layers "F.Cu" "F.Paste" "F.Mask")
-      (net 3 "csb1") (pintype "stereo"))
+      (net 6 "vcc") (pintype "stereo"))
     (pad "15" smd rect (at 1.2 1.5 270) (size 0.25 0.8) (layers "F.Cu" "F.Paste" "F.Mask")
-      (net 2 "sdo2") (pintype "stereo"))
+      (net 3 "sdo1") (pintype "stereo"))
     (pad "16" smd rect (at 0 1.91) (size 0.25 0.8) (layers "F.Cu" "F.Paste" "F.Mask")
       (net 1 "int1") (pintype "stereo"))
@@
   (segment (start 161.652177 94.035624) (end 161.561553 93.945) (width 0.25) (layer "F.Cu") (net 6))
   (segment (start 156.856993 92.480233) (end 156.563308 92.480233) (width 0.25) (layer "F.Cu") (net 6))
+  (segment (start 160.995 95.395) (end 160.995 93.995) (width 0.25) (layer "F.Cu") (net 6))
   (segment (start 158.545 94.945) (end 159.545 93.945) (width 0.25) (layer "F.Cu") (net 6))
-  (segment (start 161.561553 93.945) (end 160.27 93.945) (width 0.25) (layer "F.Cu") (net 6))
   (segment (start 158.980259 93.563914) (end 158.980259 93.573032) (width 0.25) (layer "F.Cu") (net 6))
   (segment (start 158.980259 93.573032) (end 159.352227 93.945) (width 0.25) (layer "F.Cu") (net 6))
   (segment (start 157.87 92.945) (end 158.361345 92.945) (width 0.25) (layer "F.Cu") (net 6))
   (segment (start 157.32176 92.945) (end 156.856993 92.480233) (width 0.25) (layer "F.Cu") (net 6))
+  (segment (start 160.655 93.945) (end 160.27 93.945) (width 0.25) (layer "F.Cu") (net 6))
+  (segment (start 160.945 95.445) (end 160.995 95.395) (width 0.25) (layer "F.Cu") (net 6))
+  (segment (start 160.945 93.945) (end 160.655 93.945) (width 0.25) (layer "F.Cu") (net 6))
+  (segment (start 160.27 95.445) (end 160.945 95.445) (width 0.25) (layer "F.Cu") (net 6))
   (segment (start 158.361345 92.945) (end 158.980259 93.563914) (width 0.25) (layer "F.Cu") (net 6))
   (segment (start 159.352227 93.945) (end 160.27 93.945) (width 0.25) (layer "F.Cu") (net 6))
   (segment (start 157.87 92.945) (end 157.32176 92.945) (width 0.25) (layer "F.Cu") (net 6))
+  (segment (start 161.561553 93.945) (end 160.655 93.945) (width 0.25) (layer "F.Cu") (net 6))
+  (segment (start 160.995 93.995) (end 160.945 93.945) (width 0.25) (layer "F.Cu") (net 6))
+  (segment (start 158.598297 95.445) (end 157.87 95.445) (width 0.25) (layer "F.Cu") (net 9))
+  (segment (start 160.995 96.395) (end 159.545 96.395) (width 0.25) (layer "F.Cu") (net 9))
   (segment (start 157.87 93.445) (end 156.568075 93.445) (width 0.25) (layer "F.Cu") (net 9))
-  (segment (start 159.545 95.72451) (end 159.26549 95.445) (width 0.25) (layer "F.Cu") (net 9))
+  (segment (start 159.545 96.395) (end 159.52 96.37) (width 0.25) (layer "F.Cu") (net 9))
   (segment (start 156.568075 93.445) (end 156.563308 93.440233) (width 0.25) (layer "F.Cu") (net 9))
+  (segment (start 161.652177 95.737823) (end 160.995 96.395) (width 0.25) (layer "F.Cu") (net 9))
   (segment (start 157.87 94.445) (end 157.195 94.445) (width 0.25) (layer "F.Cu") (net 9))
-  (segment (start 159.545 96.395) (end 159.545 95.72451) (width 0.25) (layer "F.Cu") (net 9))
-  (segment (start 159.26549 95.445) (end 157.87 95.445) (width 0.25) (layer "F.Cu") (net 9))
+  (segment (start 159.52 96.37) (end 159.52 95.63) (width 0.25) (layer "F.Cu") (net 9))
   (segment (start 157.195 94.445) (end 157.145 94.495) (width 0.25) (layer "F.Cu") (net 9))
   (segment (start 156.563308 93.440233) (end 157.145 94.021925) (width 0.25) (layer "F.Cu") (net 9))
@@
   (segment (start 157.145 94.495) (end 157.145 95.395) (width 0.25) (layer "F.Cu") (net 9))
   (segment (start 157.145 94.021925) (end 157.145 94.495) (width 0.25) (layer "F.Cu") (net 9))
-  (segment (start 161.652177 95.737823) (end 160.995 96.395) (width 0.25) (layer "F.Cu") (net 9))
-  (segment (start 160.995 96.395) (end 159.545 96.395) (width 0.25) (layer "F.Cu") (net 9))
+  (segment (start 158.783297 95.63) (end 158.598297 95.445) (width 0.25) (layer "F.Cu") (net 9))
+  (segment (start 159.52 95.63) (end 158.783297 95.63) (width 0.25) (layer "F.Cu") (net 9))
   (segment (start 161.652177 94.995624) (end 161.652177 95.737823) (width 0.25) (layer "F.Cu") (net 9))
   (segment (start 157.195 95.445) (end 157.87 95.445) (width 0.25) (layer "F.Cu") (net 9))
